Commit message: first commit

File: scout_description/urdf/scout_mini.urdf.xacro (robot description, xacro)
@@ -6,4 +6,7 @@
     <!-- Variables -->
     <xacro:property name="M_PI" value="3.14159"/>
+    <material name="white">
+        <color rgba="1 1 1 1"/>
+    </material>
     <!-- Vehicle Geometries -->
     <xacro:property name="base_x_size" value="0.6200000" />
@@ -20,5 +23,5 @@
             <origin
                     xyz="0 0 0"
-                    rpy="1.5707 0 -1.5707" />
+                    rpy="${pi/2} 0 -${pi/2}" />
             <geometry>
                 <mesh filename="package://scout_description/meshes/scout_mini_base_link.dae" />
@@ -28,5 +31,5 @@
             <origin
                     xyz="0 0 0"
-                    rpy="1.5707 0 -1.5707" />
+                    rpy="${pi/2} 0 -${pi/2}" />
           <geometry>
             <mesh
@@ -46,4 +49,20 @@
         <parent link="base_link" />
         <child link="inertial_link" />
+    </joint>
+<!-- Outer S1 -->
+    <link name="ousterS1">
+        <visual>
+            <origin xyz="0 0 0" rpy="0 0 0"/> <!-- Adjust this to set the position and orientation -->
+            <geometry>
+            <mesh filename="package://scout_description/meshes/mid-360-asm.stl" scale="1 1 1"/>
+            </geometry>
+            <material name="white"/>
+        </visual>
+    </link>
+    <!-- Joint connecting RPLIDAR to a part of the robot, e.g., base_link -->
+    <joint name="ousterS1_joint" type="fixed">
+        <parent link="base_link"/>
+        <child link="ousterS1"/>
+        <origin xyz="0.0  0.0  0.3" rpy="0 0 0"/> <!-- Change this to adjust the position -->
     </joint>
     <!-- Scout wheel macros -->

Commit message: robot_description_done

File: scout_description/urdf/scout_mini.urdf.xacro (robot description, xacro)
@@ -50,4 +50,20 @@
         <child link="inertial_link" />
     </joint>
+<!-- Aluminum stand-->
+    <link name="Aluminum_stand">
+        <visual>
+            <origin xyz="0 0 0" rpy="0 0 0"/> <!-- Adjust this to set the position and orientation -->
+            <geometry>
+            <mesh filename="package://scout_description/meshes/scoutmini_stand.stl" scale="1 1 1"/>
+            </geometry>
+            <material name="white"/>
+        </visual>
+    </link>
+    <!-- Joint connecting RPLIDAR to a part of the robot, e.g., base_link -->
+    <joint name="Aluminum_stand_joint" type="fixed">
+        <parent link="base_link"/>
+        <child link="Aluminum_stand"/>
+        <origin xyz="0.0  0.0  0.155 " rpy="0 0 0"/> <!-- Change this to adjust the position -->
+    </joint>
 <!-- Outer S1 -->
     <link name="ousterS1">
@@ -55,5 +71,5 @@
             <origin xyz="0 0 0" rpy="0 0 0"/> <!-- Adjust this to set the position and orientation -->
             <geometry>
-            <mesh filename="package://scout_description/meshes/mid-360-asm.stl" scale="1 1 1"/>
+            <mesh filename="package://scout_description/meshes/untitled.stl" scale="1 1 1"/>
             </geometry>
             <material name="white"/>
@@ -62,7 +78,7 @@
     <!-- Joint connecting RPLIDAR to a part of the robot, e.g., base_link -->
     <joint name="ousterS1_joint" type="fixed">
-        <parent link="base_link"/>
+        <parent link="Aluminum_stand"/>
         <child link="ousterS1"/>
-        <origin xyz="0.0  0.0  0.3" rpy="0 0 0"/> <!-- Change this to adjust the position -->
+        <origin xyz="-0.0254  0.0  0.215" rpy="0 0 0"/> <!-- Change this to adjust the position -->
     </joint>
     <!-- Scout wheel macros -->

Commit message: ouster_link

File: scout_description/urdf/scout_mini.urdf.xacro (robot description, xacro)
@@ -67,5 +67,5 @@
     </joint>
 <!-- Outer S1 -->
-    <link name="ousterS1">
+    <link name="os_sensor">
         <visual>
             <origin xyz="0 0 0" rpy="0 0 0"/> <!-- Adjust this to set the position and orientation -->

Commit message: cmd_vel_type_changed

File: scout_description/urdf/scout_mini.urdf.xacro (robot description, xacro)
@@ -79,5 +79,5 @@
     <joint name="ousterS1_joint" type="fixed">
         <parent link="Aluminum_stand"/>
-        <child link="ousterS1"/>
+        <child link="os_sensor"/>
         <origin xyz="-0.0254  0.0  0.215" rpy="0 0 0"/> <!-- Change this to adjust the position -->
     </joint>
